File: KiCAD/BME280_KiCAD/BME280_KiCAD.kicad_sch (KiCad schematic)
At the start: 21 parts, among them Q1 2N7000, Q2 2N7000, Q3 2N7000, U1 D148K, U2 ESP32-S3-DevKitC, U3 D148K, U4 D148K

Commit message: added code folder with a template file and the file where the full code will be.
Parts:
- added U5: 2652, BME280_local:MODULE_2652, symbol BME280_local:2652
Connections:
- net GND: now also U5.3 (GND)
- net SCL: now also U5.4 (SCK/SCL)
- net SDA: now also U5.6 (SDI/SDA)
- net VCC (3.3V): now also U5.2 (3VO), U5.5 (SDO)
- no-connect marks 28 -> 30
