File: KiCAD/BME280_KiCAD/BME280_KiCAD.kicad_sch (KiCad schematic)
At the start: 22 parts, among them Q1 2N7000, Q2 2N7000, Q3 2N7000, U1 D148K, U2 ESP32-S3-DevKitC, U3 D148K, U4 D148K, U5 2652

Commit message: made I2C oled display work without library, next time will use adafruit library
Parts:
- removed Q1, Q2, Q3: 2N7000, Package_TO_SOT_THT:TO-92_Inline_Wide, symbol Transistor_FET:2N7000
- added Q4, Q5, Q6: IRLZ44N, Package_TO_SOT_THT:TO-220-3_Vertical, symbol Transistor_FET:IRLZ44N
- U2: footprint esp32_local:ESP32-S3-DevKitC -> esp32:ESP32-S3
Connections:
- net GND: now also Q4.3 (S), Q5.3 (S), Q6.3 (S)
- net at R10.2, R9.2: now also Q4.1 (G)
- net at R13.2, R14.2: now also Q6.1 (G)
- net at U4.8 (CC): now also Q6.2 (D)
- net at R11.2, R12.2: now also Q5.1 (G)
- net at U3.8 (CC): now also Q5.2 (D)
- net at U1.8 (CC): now also Q4.2 (D)
